File: Kicad/Pulseox/Pulseox.sch (KiCad schematic (older format))
At the start: 48 parts, among them IC2 MCP1700T-3002E/TT, T3V TEST, U1 TSL13T, U2 MCP1640T-I/CHY, U4 STM32F030F4P6, U5 Button, U6 Button, U7 PIEZZO, X1 CONN_01X29

Commit message: Updated schematic
Parts:
- added SJ1: SJ1, Connectors:GS2, symbol GS2
Connections:
- net 3V0: now also SJ1.2 (G2); no longer U4.1 (BOOT0)
- new net: SJ1.1 (G1), U4.1 (BOOT0)
Other:
- note added: "Control\n"
- note added: "IRNAS\nInstitute for development of advanced \naplied systems Rače"
- note added: "Pulseox"
- note removed: "Controll"
